Commit message: feat: add 3d model

File: cybership_description/urdf/cybership_enterprise1_base.urdf (robot description, URDF)
Before this commit: robot cybership_enterprise_1, 5 links, 4 joints
Links:
- link base_link: geometry visual mesh filename=package://cybership_description/meshes/cs_enterprise_1_mode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 scale=0.01 0.01 0.01

Commit message: feat: simulation migration

File: cybership_description/urdf/cybership_enterprise1_base.urdf (robot description, URDF)
Before this commit: robot cybership_enterprise_1, 5 links, 4 joints
Joints:
- joint bow_tunnel_thruster_joint: origin xyz=0.3875 0 -0.05 rpy=0 0 0 -> xyz=0.3875 0 -0.05 rpy=0 0 1.5707963267948966
