Commit message: fix: simulator

File: cybership_description/urdf/model/enterprise/base.urdf.xacro (robot description, xacro)
@@ -14,6 +14,4 @@
             </geometry>
         </visual>
-    </link>
-    <link name="imu_link">
     </link>
     <link name="stern_port_thruster_link"/>
@@ -35,4 +33,5 @@
         <origin xyz="0.3875 0 -0.05" rpy="0 0 1.5707963267948966"/>
     </joint>
+    <link name="imu_link"></link>
     <joint name="imu_joint" type="fixed">
         <parent link="base_link"/>
@@ -40,3 +39,9 @@
         <origin xyz="0.4 0 0.1" rpy="0 0 0"/>
     </joint>
+    <link name="mocap_link"></link>
+    <joint name="mocap_link_joint" type="fixed">
+        <parent link="base_link"/>
+        <child link="mocap_link"/>
+        <origin xyz="0.0 0.0 0.0" rpy="0.0 3.14159265358979 1.5707963267948966"/>
+    </joint>
 </robot>

Commit message: feat: wowhohohow so much have changed. absolutely no idea how to write them now.

File: cybership_description/urdf/model/enterprise/base.urdf.xacro (robot description, xacro)
@@ -1,4 +1,10 @@
 <?xml version="1.0"?>
 <robot xmlns:xacro="http://www.ros.org/wiki/xacro" name="cybership_enterprise">
+    <!-- TODO: Fix thruster frame orientations and coordinate systems
+         - Thruster frames are not correctly oriented according to their actual thrust directions
+         - Missing base_link_ned link for proper NED (North-East-Down) coordinate frame convention
+         - Thruster positions and orientations need to be verified against actual vessel geometry
+         - Consider adding proper coordinate frame transformations for marine robotics conventions
+    -->
     <link name="base_link">
         <visual>

File: cybership_description/urdf/model/voyager/base.urdf.xacro (robot description, xacro)
@@ -3,9 +3,5 @@
     <link name="base_link">
         <visual>
-            <!-- <origin
-                xyz="0.05 0.0 0.05"
-                rpy="1.5707963267948966 0.0 1.5707963267948966"
-            /> -->
-            !-- <origin
+            <origin
                 xyz="0.0 0.0 0.0"
                 rpy="0.0 0.0 3.141592653589793"
