Commit message: feat: improve launch include structure add robot description

File: cybership_description/urdf/model/voyager/base.urdf.xacro (robot description, xacro)
@@ -1,14 +1,12 @@
 <?xml version="1.0"?>
 <robot xmlns:xacro="http://www.ros.org/wiki/xacro" name="cybership_voyager">
-    <link name="base_link">
-    </link>
-    <link name="base_link_ned"></link>
-    <joint name="base_link_transform" type="fixed">
+    <link name="base_link"></link>
+    <link name="mocap_link"></link>
+    <joint name="mocap_link_joint" type="fixed">
         <parent link="base_link"/>
-        <child link="base_link_ned"/>
-        <origin xyz="0.0 0.0 0.0" rpy="0.0 0.0 1.5707963267948966"/>
+        <child link="mocap_link"/>
+        <origin xyz="0.0 0.0 0.0" rpy="0.0 3.14159265358979 1.5707963267948966"/>
     </joint>
-    <link name="imu_link">
-    </link>
+    <link name="imu_link"></link>
     <joint name="imu_joint" type="fixed">
         <parent link="base_link"/>

Commit message: feat: add localization

File: cybership_description/urdf/model/voyager/base.urdf.xacro (robot description, xacro)
@@ -6,5 +6,5 @@
         <parent link="base_link"/>
         <child link="mocap_link"/>
-        <origin xyz="0.0 0.0 0.0" rpy="0.0 3.14159265358979 1.5707963267948966"/>
+        <origin xyz="0.0 0.0 0.3" rpy="0.0 3.14159265358979 1.5707963267948966"/>
     </joint>
     <link name="imu_link"></link>

Commit message: feat: add control allocation

File: cybership_description/urdf/model/voyager/base.urdf.xacro (robot description, xacro)
@@ -12,5 +12,23 @@
         <parent link="base_link"/>
         <child link="imu_link"/>
-        <origin xyz="-0.1 0 0.1" rpy="0 0 0"/>
+        <origin xyz="-0.1 0 0.1" rpy="0 0 3.14159265358979"/>
+    </joint>
+    <link name="stern_port_thruster_link"/>
+    <joint name="base_stern_port_thruster_joint" type="fixed">
+        <parent link="base_link"/>
+        <child link="stern_port_thruster_link"/>
+        <origin xyz="-0.4574 0.055 -0.1" rpy="0 0 0"/>
+    </joint>
+    <link name="stern_starboard_thruster_link"/>
+    <joint name="stern_starboard_thruster_joint" type="fixed">
+        <parent link="base_link"/>
+        <child link="stern_starboard_thruster_link"/>
+        <origin xyz="-0.4574 -0.055 -0.1" rpy="0 0 0"/>
+    </joint>
+    <link name="bow_tunnel_thruster_link"/>
+    <joint name="bow_tunnel_thruster_joint" type="fixed">
+        <parent link="base_link"/>
+        <child link="bow_tunnel_thruster_link"/>
+        <origin xyz="0.3875 0 -0.05" rpy="0 0 1.5707963267948966"/>
     </joint>
 </robot>

Commit message: chore: apply modifications

File: cybership_description/urdf/model/voyager/base.urdf.xacro (robot description, xacro)
@@ -12,5 +12,5 @@
         <parent link="base_link"/>
         <child link="imu_link"/>
-        <origin xyz="-0.1 0 0.1" rpy="0 0 3.14159265358979"/>
+        <origin xyz="-0.1 0 0.1" rpy="3.14159265358979 0.0 0.0"/>
     </joint>
     <link name="stern_port_thruster_link"/>

Commit message: fix: fix them all transformations, omg, there are so many!

File: cybership_description/urdf/model/voyager/base.urdf.xacro (robot description, xacro)
@@ -19,4 +19,10 @@
         </visual>
     </link>
+    <link name="base_link_ned"/>
+    <joint name="base_link_to_ned" type="fixed">
+        <parent link="base_link_ned"/>
+        <child link="base_link"/>
+        <origin xyz="0 0 0" rpy="-3.1415926 0 0.0"/>
+    </joint>
     <link name="mocap_link"></link>
     <joint name="mocap_link_joint" type="fixed">
@@ -35,5 +41,5 @@
         <parent link="base_link" />
         <child link="stern_port_thruster_link" />
-        <origin xyz="-0.4574 0.055 -0.1" rpy="0 0 0" />
+        <origin xyz="-0.4574 0.055 -0.1" rpy="3.14159265358979 0 0.0" />
     </joint>
     <link name="stern_starboard_thruster_link" />
@@ -41,5 +47,5 @@
         <parent link="base_link" />
         <child link="stern_starboard_thruster_link" />
-        <origin xyz="-0.4574 -0.055 -0.1" rpy="0 0 0" />
+        <origin xyz="-0.4574 -0.055 -0.1" rpy="3.14159265358979 0 0" />
     </joint>
     <link name="bow_tunnel_thruster_link" />
@@ -47,5 +53,5 @@
         <parent link="base_link" />
         <child link="bow_tunnel_thruster_link" />
-        <origin xyz="0.3875 0 -0.05" rpy="0 0 1.5707963267948966" />
+        <origin xyz="0.3875 0 -0.05" rpy="3.14159265358979 0 -1.5707963267948966" />
     </joint>
 </robot>

Commit message: fix: localization issues

File: cybership_description/urdf/model/voyager/base.urdf.xacro (robot description, xacro)
@@ -17,12 +17,13 @@
     <link name="base_link_ned"/>
     <joint name="base_link_to_ned" type="fixed">
+        <child link="base_link"/>
         <parent link="base_link_ned"/>
-        <child link="base_link"/>
         <origin xyz="0 0 0" rpy="-3.1415926 0 0.0"/>
     </joint>
     <link name="mocap_link"></link>
     <joint name="mocap_link_joint" type="fixed">
-        <parent link="base_link" />
+        <parent link="base_link_ned" />
         <child link="mocap_link" />
+        <!-- <origin xyz="0.0 0.0 0.3" rpy="0.0 0.0 0.0" /> -->
         <origin xyz="0.0 0.0 0.3" rpy="0.0 3.14159265358979 1.5707963267948966" />
     </joint>
