Commit message: feat: add drillship and enterprise simulation

File: cybership_description/urdf/model/drillship/base.urdf.xacro (robot description, xacro)
@@ -1,4 +1,36 @@
 <?xml version="1.0"?>
-<robot xmlns:xacro="http://www.ros.org/wiki/xacro" name="cybership_drillship">
+<robot xmlns:xacro="http://www.ros.org/wiki/xacro" name="cybership_voyager">
     <link name="base_link"></link>
+    <link name="mocap_link"></link>
+    <joint name="mocap_link_joint" type="fixed">
+        <parent link="base_link" />
+        <child link="mocap_link" />
+        <origin xyz="0.0 0.0 0.3" rpy="0.0 3.14159265358979 1.5707963267948966" />
+    </joint>
+    <link name="imu_link"></link>
+    <joint name="imu_joint" type="fixed">
+        <parent link="base_link" />
+        <child link="imu_link" />
+        <origin xyz="-0.1 0 0.1" rpy="3.14159265358979 0.0 0.0" />
+    </joint>
+    <xacro:macro name="thruster" params="thruster_name origin_xyz origin_rpy">
+        <link name="${thruster_name}_link" />
+        <joint name="${thruster_name}_joint" type="fixed">
+            <parent link="base_link" />
+            <child link="${thruster_name}_link" />
+            <origin xyz="${origin_xyz}" rpy="${origin_rpy}" />
+        </joint>
+    </xacro:macro>
+    <xacro:thruster thruster_name="bow_port_azimuth" origin_xyz="0.9344 -0.11 -0.1"
+        origin_rpy="0 0 0" />
+    <xacro:thruster thruster_name="bow_center_azimuth" origin_xyz="1.0678 0.0 -0.01"
+        origin_rpy="0 0 0" />
+    <xacro:thruster thruster_name="bow_starboard_azimuth" origin_xyz="0.9344 0.11 -0.1"
+        origin_rpy="0 0 0" />
+    <xacro:thruster thruster_name="aft_port_azimuth" origin_xyz="-0.9911 -0.1644 -0.1"
+        origin_rpy="0 0 0" />
+    <xacro:thruster thruster_name="aft_center_azimuth" origin_xyz="-1.1644 0.0 -0.01"
+        origin_rpy="0 0 0" />
+    <xacro:thruster thruster_name="aft_starboard_azimuth" origin_xyz="-0.9911 0.1644 -0.1"
+        origin_rpy="0 0 0" />
 </robot>

Commit message: feat: add dp for drillship

File: cybership_description/urdf/model/drillship/base.urdf.xacro (robot description, xacro)
@@ -1,5 +1,6 @@
 <?xml version="1.0"?>
 <robot xmlns:xacro="http://www.ros.org/wiki/xacro" name="cybership_voyager">
-    <link name="base_link"></link>
+    <link name="base_link">
+    </link>
     <link name="mocap_link"></link>
     <joint name="mocap_link_joint" type="fixed">
@@ -22,15 +23,15 @@
         </joint>
     </xacro:macro>
-    <xacro:thruster thruster_name="bow_port_azimuth" origin_xyz="0.9344 -0.11 -0.1"
+    <xacro:thruster thruster_name="bow_port_thruster" origin_xyz="0.9344 -0.11 -0.1"
         origin_rpy="0 0 0" />
-    <xacro:thruster thruster_name="bow_center_azimuth" origin_xyz="1.0678 0.0 -0.1"
+    <xacro:thruster thruster_name="bow_center_thruster" origin_xyz="1.0678 0.0 -0.1"
         origin_rpy="0 0 0" />
-    <xacro:thruster thruster_name="bow_starboard_azimuth" origin_xyz="0.9344 0.11 -0.1"
+    <xacro:thruster thruster_name="bow_starboard_thruster" origin_xyz="0.9344 0.11 -0.1"
         origin_rpy="0 0 0" />
-    <xacro:thruster thruster_name="aft_port_azimuth" origin_xyz="-0.9911 -0.1644 -0.1"
+    <xacro:thruster thruster_name="aft_port_thruster" origin_xyz="-0.9911 -0.1644 -0.1"
         origin_rpy="0 0 0" />
-    <xacro:thruster thruster_name="aft_center_azimuth" origin_xyz="-1.1644 0.0 -0.1"
+    <xacro:thruster thruster_name="aft_center_thruster" origin_xyz="-1.1644 0.0 -0.1"
         origin_rpy="0 0 0" />
-    <xacro:thruster thruster_name="aft_starboard_azimuth" origin_xyz="-0.9911 0.1644 -0.1"
+    <xacro:thruster thruster_name="aft_starboard_thruster" origin_xyz="-0.9911 0.1644 -0.1"
         origin_rpy="0 0 0" />
 </robot>

File: cybership_description/urdf/model/enterprise/base.urdf.xacro (robot description, xacro)
@@ -9,39 +9,39 @@
             <geometry>
                 <mesh
-                    filename="package://cybership_description/meshes/cs_enterprise_1_model_lowpoly.dae"
+                    filename="package://cybership_description/meshes/enterprise/model.stl"
                     scale="0.01 0.01 0.01"
-                    />
+                />
             </geometry>
         </visual>
     </link>
-    <link name="stern_port_thruster_link"/>
+    <link name="stern_port_thruster_link" />
     <joint name="base_stern_port_thruster_joint" type="fixed">
-        <parent link="base_link"/>
-        <child link="stern_port_thruster_link"/>
-        <origin xyz="-0.4574 0.055 -0.1" rpy="0 0 0"/>
+        <parent link="base_link" />
+        <child link="stern_port_thruster_link" />
+        <origin xyz="-0.4574 0.055 -0.1" rpy="0 0 0" />
     </joint>
-    <link name="stern_starboard_thruster_link"/>
+    <link name="stern_starboard_thruster_link" />
     <joint name="stern_starboard_thruster_joint" type="fixed">
-        <parent link="base_link"/>
-        <child link="stern_starboard_thruster_link"/>
-        <origin xyz="-0.4574 -0.055 -0.1" rpy="0 0 0"/>
+        <parent link="base_link" />
+        <child link="stern_starboard_thruster_link" />
+        <origin xyz="-0.4574 -0.055 -0.1" rpy="0 0 0" />
     </joint>
-    <link name="bow_tunnel_thruster_link"/>
+    <link name="bow_tunnel_thruster_link" />
     <joint name="bow_tunnel_thruster_joint" type="fixed">
-        <parent link="base_link"/>
-        <child link="bow_tunnel_thruster_link"/>
-        <origin xyz="0.3875 0 -0.05" rpy="0 0 1.5707963267948966"/>
+        <parent link="base_link" />
+        <child link="bow_tunnel_thruster_link" />
+        <origin xyz="0.3875 0 -0.05" rpy="0 0 1.5707963267948966" />
     </joint>
     <link name="imu_link"></link>
     <joint name="imu_joint" type="fixed">
-        <parent link="base_link"/>
-        <child link="imu_link"/>
-        <origin xyz="0.4 0 0.1" rpy="0 0 0"/>
+        <parent link="base_link" />
+        <child link="imu_link" />
+        <origin xyz="0.4 0 0.1" rpy="0 0 0" />
     </joint>
     <link name="mocap_link"></link>
     <joint name="mocap_link_joint" type="fixed">
-        <parent link="base_link"/>
-        <child link="mocap_link"/>
-        <origin xyz="0.0 0.0 0.0" rpy="0.0 3.14159265358979 1.5707963267948966"/>
+        <parent link="base_link" />
+        <child link="mocap_link" />
+        <origin xyz="0.0 0.0 0.0" rpy="0.0 3.14159265358979 1.5707963267948966" />
     </joint>
 </robot>

File: cybership_description/urdf/model/voyager/base.urdf.xacro (robot description, xacro)
@@ -1,34 +1,51 @@
 <?xml version="1.0"?>
 <robot xmlns:xacro="http://www.ros.org/wiki/xacro" name="cybership_voyager">
-    <link name="base_link"></link>
+    <link name="base_link">
+        <visual>
+            <!-- <origin
+                xyz="0.05 0.0 0.05"
+                rpy="1.5707963267948966 0.0 1.5707963267948966"
+            /> -->
+            !-- <origin
+                xyz="0.0 0.0 0.0"
+                rpy="0.0 0.0 3.141592653589793"
+            />
+            <geometry>
+                <mesh
+                    filename="package://cybership_description/meshes/voyager/model.stl"
+                    scale="1.0 1.0 1.0"
+                />
+            </geometry>
+        </visual>
+    </link>
     <link name="mocap_link"></link>
     <joint name="mocap_link_joint" type="fixed">
-        <parent link="base_link"/>
-        <child link="mocap_link"/>
-        <origin xyz="0.0 0.0 0.3" rpy="0.0 3.14159265358979 1.5707963267948966"/>
+        <parent link="base_link" />
+        <child link="mocap_link" />
+        <origin xyz="0.0 0.0 0.3" rpy="0.0 3.14159265358979 1.5707963267948966" />
     </joint>
     <link name="imu_link"></link>
     <joint name="imu_joint" type="fixed">
-        <parent link="base_link"/>
-        <child link="imu_link"/>
-        <origin xyz="-0.1 0 0.1" rpy="3.14159265358979 0.0 0.0"/>
+        <parent link="base_link" />
+        <child link="imu_link" />
+        <origin xyz="-0.1 0 0.1" rpy="3.14159265358979 0.0 0.0" />
     </joint>
-    <link name="stern_port_thruster_link"/>
+    <link name="stern_port_thruster_link" />
     <joint name="base_stern_port_thruster_joint" type="fixed">
-        <parent link="base_link"/>
-        <child link="stern_port_thruster_link"/>
-        <origin xyz="-0.4574 0.055 -0.1" rpy="0 0 0"/>
+        <parent link="base_link" />
+        <child link="stern_port_thruster_link" />
+        <origin xyz="-0.4574 0.055 -0.1" rpy="0 0 0" />
     </joint>
-    <link name="stern_starboard_thruster_link"/>
+    <link name="stern_starboard_thruster_link" />
     <joint name="stern_starboard_thruster_joint" type="fixed">
-        <parent link="base_link"/>
-        <child link="stern_starboard_thruster_link"/>
-        <origin xyz="-0.4574 -0.055 -0.1" rpy="0 0 0"/>
+        <parent link="base_link" />
+        <child link="stern_starboard_thruster_link" />
+        <origin xyz="-0.4574 -0.055 -0.1" rpy="0 0 0" />
     </joint>
-    <link name="bow_tunnel_thruster_link"/>
+    <link name="bow_tunnel_thruster_link" />
     <joint name="bow_tunnel_thruster_joint" type="fixed">
-        <parent link="base_link"/>
-        <child link="bow_tunnel_thruster_link"/>
-        <origin xyz="0.3875 0 -0.05" rpy="0 0 1.5707963267948966"/>
+        <parent link="base_link" />
+        <child link="bow_tunnel_thruster_link" />
+        <origin xyz="0.3875 0 -0.05" rpy="0 0 1.5707963267948966" />
     </joint>
 </robot>

Commit message: feat: add drillship

File: cybership_description/urdf/model/drillship/base.urdf.xacro (robot description, xacro)
@@ -3,7 +3,13 @@
     <link name="base_link">
     </link>
+    <link name="base_link_ned"/>
+    <joint name="base_link_to_ned" type="fixed">
+        <child link="base_link"/>
+        <parent link="base_link_ned"/>
+        <origin xyz="0 0 0" rpy="-3.1415926 0 0.0"/>
+    </joint>
     <link name="mocap_link"></link>
     <joint name="mocap_link_joint" type="fixed">
-        <parent link="base_link" />
+        <parent link="base_link_ned" />
         <child link="mocap_link" />
         <origin xyz="0.0 0.0 0.3" rpy="0.0 3.14159265358979 1.5707963267948966" />

Commit message: fix: position controller and localization for drillship

File: cybership_description/urdf/model/drillship/base.urdf.xacro (robot description, xacro)
@@ -13,4 +13,5 @@
         <parent link="base_link_ned" />
         <child link="mocap_link" />
+        <!-- <origin xyz="0.0 0.0 0.3" rpy="0.0 0.0 0.0" /> -->
         <origin xyz="0.0 0.0 0.3" rpy="0.0 3.14159265358979 1.5707963267948966" />
     </joint>

Commit message: feat: add multi vehicle sim support

File: cybership_description/urdf/model/drillship/base.urdf.xacro (robot description, xacro)
@@ -2,4 +2,16 @@
 <robot xmlns:xacro="http://www.ros.org/wiki/xacro" name="cybership_voyager">
     <link name="base_link">
+        <visual>
+            <origin
+                xyz="0.0 0.0 0.0"
+                rpy="0.0 0.0 0.0"
+            />
+            <geometry>
+                <mesh
+                    filename="package://cybership_description/meshes/drillship/model.stl"
+                    scale="1.0 1.0 1.0"
+                />
+            </geometry>
+        </visual>
     </link>
     <link name="base_link_ned"/>

Commit message: fix: transforms

File: cybership_description/urdf/model/drillship/base.urdf.xacro (robot description, xacro)
@@ -37,5 +37,5 @@
         <link name="${thruster_name}_link" />
         <joint name="${thruster_name}_joint" type="fixed">
-            <parent link="base_link" />
+            <parent link="base_link_ned" />
             <child link="${thruster_name}_link" />
             <origin xyz="${origin_xyz}" rpy="${origin_rpy}" />

File: cybership_description/urdf/model/voyager/base.urdf.xacro (robot description, xacro)
@@ -30,8 +30,32 @@
     <link name="imu_link"></link>
     <joint name="imu_joint" type="fixed">
-        <parent link="base_link" />
+        <parent link="base_link_ned" />
         <child link="imu_link" />
-        <origin xyz="-0.1 0 0.1" rpy="3.14159265358979 0.0 0.0" />
+        <origin xyz="-0.1 0 0.1" rpy="0.0 0.0 0.0" />
     </joint>
+    <xacro:macro name="thruster" params="thruster_name origin_xyz origin_rpy">
+        <link name="${thruster_name}_link" />
+        <joint name="${thruster_name}_joint" type="fixed">
+            <parent link="base_link_ned" />
+            <child link="${thruster_name}_link" />
+            <origin xyz="${origin_xyz}" rpy="${origin_rpy}" />
+        </joint>
+    </xacro:macro>
+    <xacro:thruster
+        thruster_name="stern_port_thruster"
+        origin_xyz="-0.4574 -0.055 0.1"
+        origin_rpy="0 0 0"
+    />
+    <xacro:thruster
+        thruster_name="stern_starboard_thruster"
+        origin_xyz="-0.4574 0.055 0.1"
+        origin_rpy="0 0 0"
+    />
+    <xacro:thruster
+        thruster_name="bow_tunnel_thruster"
+        origin_xyz="0.3875 0 0.05"
+        origin_rpy="0 0 -1.5707963267948966"
+    />
+<!--
     <link name="stern_port_thruster_link" />
     <joint name="base_stern_port_thruster_joint" type="fixed">
@@ -51,4 +75,4 @@
         <child link="bow_tunnel_thruster_link" />
         <origin xyz="0.3875 0 -0.05" rpy="3.14159265358979 0 -1.5707963267948966" />
-    </joint>
+    </joint> -->
 </robot>
